File: 8884bt Remote Control Receiver/board/Brickster 8884bt Receiver.brd (EAGLE design)
At the start: 28.8 x 28.8 mm, 20 parts, among them J1 AVR_SPI_PRG_6NS, J2 CON_PF_SMD, J3 CON_PF_SMD, J4 CON_PF_SMD, U1 IC_ATTINY_X4A, U2 IC_DRV8833, U3 IC_RT9164A, U4 HC-06

Commit message: Update receiver to revision 3
Parts:
- removed B2, B3, B4: B_CDBHM240L-HF, brickster:MBS-2
- removed C5: 10uF, brickster:1206
- removed J2, J3, J4: CON_PF_SMD, brickster:SMD_PF
- removed LOGO2: OSHW-LOGOM, SparkFun-Aesthetics:OSHW-LOGO-M-MASK
- removed U1: IC_ATTINY_X4A, brickster:14S1
- removed U3: IC_RT9164A, brickster:SOT223
- removed U4: HC-06, brickster:BLUETOOTH_SMD
- added NCP1117ST33T3G: IC_RT9164A, brickster:SOT223
- added Q1: DMHC3025LSD-13, brickster:SO8
- added R1: 10k, brickster:0402
- added R3: 3.3k, brickster:0402
- added U5: ATtiny841, bt_avr:14SOICN
- added U6: LV8402GP-TE-L-H, codefox421-parts:VCT24
- C1: value 0.1uF -> 0.1µF; device brickster:0805 -> brickster:0402
- C2: value 10uF -> 100µF
- C3: value 0.01uF -> 10nF; device brickster:0805 -> brickster:0402
- C4: value 2.2uF -> 0.1µF; device brickster:0805 -> brickster:0402
- D1: value LED0805 -> LTST-C195TBKFKT; device brickster:0805_POL -> brickster:CHIP-LTST
- LOGO1: device SparkFun-Aesthetics:OSHW-LOGO-M-MASK -> SparkFun-Aesthetics:OSHW-LOGO-M
- R2: device brickster:0805 -> brickster:0402
- U2: value IC_DRV8833 -> HM-06; device brickster:PWP_R-PDSO-G16 -> codefox421-parts:HM-05/06/07
- moved LOGO1 18.8 mm to (3.61, 10.0)
- moved U2 16.0 mm to (7.62, 13.4), flipped to the bottom, turned to 270 degrees
- moved C1 15.1 mm to (21.6, 14.6), turned to 90 degrees
- moved C2 8.06 mm to (27.4, 14.6), flipped to the bottom
- moved R2 6.51 mm to (12.0, 8.13), flipped to the top, turned to 270 degrees
- moved D1 5.36 mm to (10.4, 8.13)
- moved C4 3.79 mm to (26.1, 18.2), flipped to the bottom, turned to 180 degrees
- moved C3 1.89 mm to (25.7, 19.5), flipped to the bottom
- moved J1 0.25 mm to (2.44, 16.8)
Connections:
- removed net BTRST: U1.10, U4.11
- removed net MISO: J1.1, U1.8
- removed net MOSI: J1.4, U1.7
- removed net N$4: D1.P$2, R2.P$2
- removed net RESET: J1.5, U1.4
- removed net SCK: J1.3, U1.9
- new net !BTRST: U2.11, U5.5
- new net !RESET: J1.5, R1.2, U5.4, U6.12, U6.16
- new net N$10: C3.2, U6.19
- new net N$11: C4.1, U6.21
- new net N$15: C3.1, U6.20
- new net N$16: J1.1, U5.8
- new net N$8: U5.13
- net 3.3V: now also NCP1117ST33T3G.2, NCP1117ST33T3G.4, R1.1, R3.2, U2.9, U5.1, U6.13; no longer U1.1, U2.1, U3.2, U3.4, U4.12
- net A01: now also U6.1; no longer B3.AC1, J3.C2, U2.2
- net A02: now also U6.2; no longer B3.AC2, J3.C1, U2.4
- net AIN1: now also U5.6, U6.15; no longer U1.2, U2.16
- net AIN2: now also J1.4, U5.7, U6.14; no longer U1.3, U2.15
- net ATRX/BTTX: now also U2.2, U5.11; no longer U1.13, U4.1
- net ATTX/BTRX: now also U2.4, U5.12; no longer U1.12, U4.2
- net B01: now also U6.5; no longer B4.AC2, J4.C2, U2.7
- net B02: now also U6.6; no longer B4.AC1, J4.C1, U2.5
- net BIN1: now also J1.3, U5.9, U6.11; no longer U1.6, U2.9
- net BIN2: now also U5.10, U6.10; no longer U1.5, U2.10
- net GND: now also C1.2, C4.2, D1.3, NCP1117ST33T3G.1, Q1.P$3, U2.12, U5.14, U6.18, U6.3, U6.4; no longer B2.-, B3.-, B4.-, C1.P$2, C4.P$1, C5.2, D1.P$1, J2.GND, J3.GND, J4.GND, U1.14, U2.13, U2.17, U2.3, U2.6, U3.1, U4.13, U4.21, U4.22
- net KEY: now also U2.16, U5.2; no longer U1.11, U4.26
- net LED: now also D1.4, R2.2, U2.15, U5.3; no longer R2.P$1, U4.24
- net N$1: now also D1.2, R3.1; no longer C3.P$2, U2.11
- net N$2: now also D1.1, R2.1; no longer C4.P$2, U2.14
- net N$3: now also U2.1, U2.3; no longer U4.3, U4.4
- net PF_C1: now also Q1.P$2, Q1.P$4, Q1.P$5; no longer B2.AC1, J2.C1
- net PF_C2: now also Q1.P$1, Q1.P$6, Q1.P$8; no longer B2.AC2, J2.C2
- net VIN: now also C1.1, NCP1117ST33T3G.3, Q1.P$7, U6.22, U6.23, U6.8, U6.9; no longer B2.+, B3.+, B4.+, C1.P$1, C3.P$1, C5.1, J2.9V, J3.9V, J4.9V, U2.12, U3.3
Routing:
- net !RESET: track 0.00 -> 32.4 mm, vias 0 -> 3
- net VIN: track 71.3 -> 49.1 mm, vias 5 -> 3
- net 3.3V: track 41.7 -> 63.3 mm, vias 1 -> 5
- net A01: track 31.8 -> 51.8 mm, vias 3 -> 1
- net MOSI: track 18.2 -> 0.00 mm, vias 2 -> 0
- net N$8: track 0.00 -> 17.7 mm, vias 0 -> 2
- net N$16: track 0.00 -> 15.7 mm
- net AIN2: track 14.6 -> 30.2 mm, vias 0 -> 1
- net KEY: track 20.9 -> 6.54 mm
- net RESET: track 14.3 -> 0.00 mm, vias 1 -> 0
- net MISO: track 13.7 -> 0.00 mm
- net BTRST: track 13.3 -> 0.00 mm, vias 1 -> 0
- net SCK: track 11.4 -> 0.00 mm
- net PF_C2: track 8.96 -> 17.6 mm, vias 0 -> 1
- net A02: track 30.9 -> 38.9 mm, vias 2 -> 1
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Other:
- board size 28.8 x 28.8 mm -> 28.8 x 20.8 mm
- board text added: "github.com/BTbricks"
- board text added: "rev. 3"
- board text removed: "github.com/codefox421/brickster"
- board text removed: "rev. 2"
