File: 8884bt Remote Control Receiver/board/Brickster 8884bt Receiver.sch (EAGLE design)
At the start: 18 parts, among them J1 AVR_SPI_PRG_6NS, J2 CON_PF_SMD, J3 CON_PF_SMD, J4 CON_PF_SMD, U1 IC_ATTINY_X4A, U2 IC_DRV8833, U3 IC_RT9164A, U4 HC-06

Commit message: Update receiver to revision 3
Parts:
- removed B2, B3, B4: B_CDBHM240L-HF, brickster:B_CDBHM240L-HF
- removed C5: 10uF, brickster:C_POL
- removed J2, J3, J4: CON_PF_SMD, brickster:CON_PF_SMD
- removed U1: IC_ATTINY_X4A, brickster:IC_ATTINY_X4A
- removed U4: HC-06, brickster:HC-06
- added Q1: DMHC3025LSD-13, brickster:IC_FET_BRIDGESO8
- added R1: 10k, brickster:R0402
- added R3: 3.3k, brickster:R0402
- added U5: ATtiny841, bt_avr:ATTINY441/841-SSU
- added U6: LV8402GP-TE-L-H, codefox421-parts:LV8402GPLV8402GP
- C1: value 0.1uF -> 0.1µF; device brickster:C0805 -> brickster:C0402
- C2: value 10uF -> 100µF
- C3: value 0.01uF -> 10nF; device brickster:C0805 -> brickster:C0402
- C4: value 2.2uF -> 0.1µF; device brickster:C0805 -> brickster:C0402
- D1: value LED0805 -> LTST-C195TBKFKT; device brickster:LED0805 -> brickster:LED_LTST_C195TBKFKT
- R2: device brickster:R0805 -> brickster:R0402; PARTNO (none) -> ERJ-3GEYJ103V
- U2: value IC_DRV8833 -> HM-06; device brickster:IC_DRV8833 -> codefox421-parts:HM-05/06/07HM-05/06/07
- renumbered U3 to NCP1117ST33T3G
Connections:
- removed net BTRST: U1.(PCINT3/T0/ADC3)PA3, U4.RESET
- removed net MISO: J1.1, U1.(PCINT5/OC1B/MISO/DO/ADC5)PA5
- removed net MOSI: J1.4, U1.(PCINT6/OC1A/SDA/MOSI/ADC6)PA6
- removed net N$4: D1.P$1, R2.2
- removed net RESET: J1.5, U1.(PCINT11/~RESET/DW)PB3
- removed net SCK: J1.3, U1.(PCINT4/T1/SCL/USCK/ADC4)PA4
- new net !BTRST: U2.!RESET, U5.(PCINT10/ADC8/CLKO/TOCC7/ICP2/RXD0)PB2
- new net !RESET: J1.5, R1.2, U5.(PCINT11/ADC9/RESET/DW)PB3, U6.AEN, U6.BEN
- new net N$10: C3.2, U6.C1L
- new net N$11: C4.1, U6.VG
- new net N$15: C3.1, U6.C1H
- new net N$16: J1.1, U5.(PCINT5/ADC5/ACO0/TOCC4/T2/TXD1/MISO)PA5
- new net N$8: U5.(PCINT0/ADC0/AREF/MISO)PA0
- net 3.3V: now also R1.1, R3.2, U2.VCC, U5.VCC, U6.VCC; no longer U1.VCC, U2.NSLEEP, U4.VDD
- net A01: now also U6.AOUT1; no longer B3.AC1, J3.P$3, U2.AOUT1
- net A02: now also U6.AOUT2; no longer B3.AC2, J3.P$2, U2.AOUT2
- net AIN1: now also U5.(PCINT7/ADC7/TOCC6/ICP1/TXD0/SS)PA7, U6.AIN1; no longer U1.(PCINT8/XTAL1/CLKI)PB0, U2.AIN1
- net AIN2: now also J1.4, U5.(PCINT6/ADC6/ACO1/TOCC5/XCK1/SDA/MOSI)PA6, U6.AIN2; no longer U1.(PCINT9/XTAL2)PB1, U2.AIN2
- net ATRX/BTTX: now also U2.UART_TX, U5.(PCINT2/ADC2/AIN01/TOCC1/RXD0/SS)PA2; no longer U1.(PCINT0/AREF/ADC0)PA0, U4.UARTTX
- net ATTX/BTRX: now also U2.UART_RX, U5.(PCINT1/ADC1/AIN00/TOCC0/TXD0/MOSI)PA1; no longer U1.(PCINT1/AIN0/ADC1)PA1, U4.UARTRX
- net B01: now also U6.BOUT1; no longer B4.AC2, J4.P$3, U2.BOUT1
- net B02: now also U6.BOUT2; no longer B4.AC1, J4.P$2, U2.BOUT2
- net BIN1: now also J1.3, U5.(PCINT4/ADC4/AIN11/TOCC3/T1/RXD1/SCL/SCK)PA4, U6.BIN1; no longer U1.(PCINT7/ICP/OC0B/ADC7)PA7, U2.BIN1
- net BIN2: now also U5.(PCINT3/ADC3/AIN10/TOCC2/T0/XCK0/SCK)PA3, U6.BIN2; no longer U1.(PCINT10/INT0/OC0A/CKOUT)PB2, U2.BIN2
- net GND: now also C4.2, D1G$1.P$2, Q1.N1S/N2S, U5.GND, U6.PGND, U6.SGND; no longer B2.-, B3.-, B4.-, C4.1, C5.-, D1.P$2, J2.P$4, J3.P$4, J4.P$4, U1.GND, U2.AISEN, U2.BISEN, U4.GND, U4.GND1, U4.GND2
- net KEY: now also U2.PIO0/KEY, U5.(PCINT8/ADC11/XTAL1/CLKI)PB0; no longer U1.(PCINT2/AIN1/ADC2)PA2, U4.PIO3
- net LED: now also D1G$2.P$2, R2.2, U2.PIO1/LED, U5.(PCINT9/ADC10/XTAL2/INT0)PB1; no longer R2.1, U4.PIO1
- net N$1: now also D1G$2.P$1, R3.1; no longer C3.2, U2.VCP
- net N$2: now also D1G$1.P$1, R2.1; no longer C4.2, U2.VINT
- net N$3: now also U2.UART_CTS, U2.UART_RTS; no longer U4.UARTCTS, U4.UARTRTS
- net PF_C1: now also Q1.N1D/P1D, Q1.N2G, Q1.P2G; no longer B2.AC1, J2.P$2
- net PF_C2: now also Q1.N1G, Q1.N2D/P2D, Q1.P1G; no longer B2.AC2, J2.P$3
- net VIN: now also Q1.P1S/P2S, U6.VM; no longer B2.+, B3.+, B4.+, C3.1, C5.+, J2.P$1, J3.P$1, J4.P$1, U2.VM
Other:
- note added: "3"
- note added: "MISO"
- note added: "MOSI"
- note added: "PWM"
- note added: "Rx"
- note added: "SCK"
- note added: "Tx"
- note removed: "2"
- moved on the sheet: C3, C4, D1G$1, J1, R2, U2
